Commit message: Rename created URDF with better joint and link naming scheme

File: crawly-urdf/crawly.urdf (robot description, URDF)
Before this commit: robot crawly, 9 links, 8 joints
Links:
- removed link link1_v131
- removed link link1_v13_11
- removed link link1_v13_21
- removed link link1_v13_31
- removed link link2_v91
- removed link link2_v9_11
- removed link link2_v9_21
- removed link link2_v9_31
- added link L1_BL1, mass 0.026073176545293626; collision mesh filename=meshes/L1_BL1.stl scale=0.001 0.001 0.001; visual mesh filename=meshes/L1_BL1.stl scale=0.001 0.001 0.001
- added link L1_BR1, mass 0.026073176545293626; collision mesh filename=meshes/L1_BR1.stl scale=0.001 0.001 0.001; visual mesh filename=meshes/L1_BR1.stl scale=0.001 0.001 0.001
- added link L1_FL1, mass 0.026073176545293626; collision mesh filename=meshes/L1_FL1.stl scale=0.001 0.001 0.001; visual mesh filename=meshes/L1_FL1.stl scale=0.001 0.001 0.001
- added link L1_FR1, mass 0.026073176545293626; collision mesh filename=meshes/L1_FR1.stl scale=0.001 0.001 0.001; visual mesh filename=meshes/L1_FR1.stl scale=0.001 0.001 0.001
- added link L2_BL1, mass 0.072990131570421; collision mesh filename=meshes/L2_BL1.stl scale=0.001 0.001 0.001; visual mesh filename=meshes/L2_BL1.stl scale=0.001 0.001 0.001
- added link L2_BR1, mass 0.072990131570421; collision mesh filename=meshes/L2_BR1.stl scale=0.001 0.001 0.001; visual mesh filename=meshes/L2_BR1.stl scale=0.001 0.001 0.001
- added link L2_FL1, mass 0.072990131570421; collision mesh filename=meshes/L2_FL1.stl scale=0.001 0.001 0.001; visual mesh filename=meshes/L2_FL1.stl scale=0.001 0.001 0.001
- added link L2_FR1, mass 0.072990131570421; collision mesh filename=meshes/L2_FR1.stl scale=0.001 0.001 0.001; visual mesh filename=meshes/L2_FR1.stl scale=0.001 0.001 0.001
- link base_link: mass 0.370797194204883 -> 0.37046418538360243
Joints:
- removed joint Revolute_1
- removed joint Revolute_2
- removed joint Revolute_3
- removed joint Revolute_4
- removed joint Revolute_5
- removed joint Revolute_6
- removed joint Revolute_7
- removed joint Revolute_8
- added joint th_1: type continuous, parent base_link, child L1_FL1, origin xyz=0.0875 0.015 0.07 rpy=0 0 0, axis -1.0 0.0 0.0
- added joint th_2: type continuous, parent base_link, child L1_FR1, origin xyz=-0.0875 0.015 0.07 rpy=0 0 0, axis 1.0 0.0 0.0
- added joint th_3: type continuous, parent base_link, child L1_BR1, origin xyz=-0.0875 0.015 -0.07 rpy=0 0 0, axis 1.0 0.0 0.0
- added joint th_4: type continuous, parent base_link, child L1_BL1, origin xyz=0.0875 0.015 -0.07 rpy=0 0 0, axis -1.0 0.0 0.0
- added joint th_5: type continuous, parent L1_FL1, child L2_FL1, origin xyz=0.0 -0.1 0.0 rpy=0 0 0, axis -1.0 -0.0 0.0
- added joint th_6: type continuous, parent L1_FR1, child L2_FR1, origin xyz=0.0 -0.1 0.0 rpy=0 0 0, axis 1.0 -0.0 -0.0
- added joint th_7: type continuous, parent L1_BR1, child L2_BR1, origin xyz=0.0 -0.1 0.0 rpy=0 0 0, axis 1.0 -0.0 -0.0
- added joint th_8: type continuous, parent L1_BL1, child L2_BL1, origin xyz=0.0 -0.1 0.0 rpy=0 0 0, axis -1.0 -0.0 0.0

Commit message: Testing Revolute Joint

File: crawly-urdf/crawly.urdf (robot description, URDF)
Before this commit: robot crawly2, 9 links, 8 joints
Joints:
- joint th_1: limit (none) -> lower=-3.14159 upper=3.14159 effort=1.18 velocity=8.05; type continuous -> revolute

Commit message: Revolute URDF

File: crawly-urdf/crawly.urdf (robot description, URDF)
Before this commit: robot crawly2, 9 links, 8 joints
Joints:
- joint th_2: limit (none) -> lower=-3.14159 upper=3.14159 effort=1.18 velocity=8.05; type continuous -> revolute
- joint th_3: limit (none) -> lower=-3.14159 upper=3.14159 effort=1.18 velocity=8.05; type continuous -> revolute
- joint th_4: limit (none) -> lower=-3.14159 upper=3.14159 effort=1.18 velocity=8.05; type continuous -> revolute
- joint th_5: limit (none) -> lower=-3.14159 upper=3.14159 effort=1.18 velocity=8.05; type continuous -> revolute
- joint th_6: limit (none) -> lower=-3.14159 upper=3.14159 effort=1.18 velocity=8.05; type continuous -> revolute
- joint th_7: limit (none) -> lower=-3.14159 upper=3.14159 effort=1.18 velocity=8.05; type continuous -> revolute
- joint th_8: limit (none) -> lower=-3.14159 upper=3.14159 effort=1.18 velocity=8.05; type continuous -> revolute
