Commit message: Big change to have a smaller crawling robot

File: main/urdf/crawly.urdf (robot description, URDF)
Before this commit: robot crawly2, 9 links, 8 joints
Links:
- link L1_BL1: mass 0.026073176545293626 -> 0.015599766964746006
- link L1_BR1: mass 0.026073176545293626 -> 0.015599766964746006
- link L1_FL1: mass 0.026073176545293626 -> 0.015599766964746006
- link L1_FR1: mass 0.026073176545293626 -> 0.015599766964746006
- link L2_BL1: mass 0.072990131570421 -> 0.063373811570421
- link L2_BR1: mass 0.072990131570421 -> 0.063373811570421
- link L2_FL1: mass 0.072990131570421 -> 0.063373811570421
- link L2_FR1: mass 0.072990131570421 -> 0.063373811570421
- link base_link: mass 0.37046418538360243 -> 0.3712874477159382
Joints:
- joint th_1: axis -1.0 0.0 0.0 -> 1.0 0.0 0.0; origin xyz=0.0875 0.015 0.07 rpy=0 0 0 -> xyz=-0.0875 0.015 -0.07 rpy=0 0 0
- joint th_2: axis 1.0 0.0 0.0 -> -1.0 0.0 -0.0; origin xyz=-0.0875 0.015 0.07 rpy=0 0 0 -> xyz=0.0875 0.015 -0.07 rpy=0 0 0
- joint th_3: axis 1.0 0.0 0.0 -> -1.0 0.0 0.0; origin xyz=-0.0875 0.015 -0.07 rpy=0 0 0 -> xyz=0.0875 0.015 0.07 rpy=0 0 0
- joint th_4: axis -1.0 0.0 0.0 -> 1.0 0.0 0.0; origin xyz=0.0875 0.015 -0.07 rpy=0 0 0 -> xyz=-0.0875 0.015 0.07 rpy=0 0 0
- joint th_5: axis -1.0 -0.0 0.0 -> 1.0 0.0 0.0; origin xyz=0.0 -0.1 0.0 rpy=0 0 0 -> xyz=0.0 -0.06 0.0 rpy=0 0 0
- joint th_6: axis 1.0 -0.0 -0.0 -> -1.0 0.0 -0.0; origin xyz=0.0 -0.1 0.0 rpy=0 0 0 -> xyz=0.0 -0.06 0.0 rpy=0 0 0
- joint th_7: axis 1.0 -0.0 -0.0 -> -1.0 0.0 0.0; origin xyz=0.0 -0.1 0.0 rpy=0 0 0 -> xyz=0.0 -0.06 0.0 rpy=0 0 0
- joint th_8: axis -1.0 -0.0 0.0 -> 1.0 0.0 0.0; origin xyz=0.0 -0.1 0.0 rpy=0 0 0 -> xyz=0.0 -0.06 0.0 rpy=0 0 0

Commit message: switch_urdf for quick test

File: main/urdf/crawly.urdf (robot description, URDF)
Before this commit: robot crawly, 9 links, 8 joints
Links:
- link L1_BL1: mass 0.015599766964746006 -> 0.026073176545293626
- link L1_BR1: mass 0.015599766964746006 -> 0.026073176545293626
- link L1_FL1: mass 0.015599766964746006 -> 0.026073176545293626
- link L1_FR1: mass 0.015599766964746006 -> 0.026073176545293626
- link L2_BL1: mass 0.063373811570421 -> 0.072990131570421
- link L2_BR1: mass 0.063373811570421 -> 0.072990131570421
- link L2_FL1: mass 0.063373811570421 -> 0.072990131570421
- link L2_FR1: mass 0.063373811570421 -> 0.072990131570421
- link base_link: mass 0.3712874477159382 -> 0.37046418538360243
Joints:
- joint th_1: axis 1.0 0.0 0.0 -> -1.0 0.0 0.0; origin xyz=-0.0875 0.015 -0.07 rpy=0 0 0 -> xyz=0.0875 0.015 0.07 rpy=0 0 0
- joint th_2: axis -1.0 0.0 -0.0 -> 1.0 0.0 0.0; origin xyz=0.0875 0.015 -0.07 rpy=0 0 0 -> xyz=-0.0875 0.015 0.07 rpy=0 0 0
- joint th_3: axis -1.0 0.0 0.0 -> 1.0 0.0 0.0; origin xyz=0.0875 0.015 0.07 rpy=0 0 0 -> xyz=-0.0875 0.015 -0.07 rpy=0 0 0
- joint th_4: axis 1.0 0.0 0.0 -> -1.0 0.0 0.0; origin xyz=-0.0875 0.015 0.07 rpy=0 0 0 -> xyz=0.0875 0.015 -0.07 rpy=0 0 0
- joint th_5: axis 1.0 0.0 0.0 -> -1.0 -0.0 0.0; origin xyz=0.0 -0.06 0.0 rpy=0 0 0 -> xyz=0.0 -0.1 0.0 rpy=0 0 0
- joint th_6: axis -1.0 0.0 -0.0 -> 1.0 -0.0 -0.0; origin xyz=0.0 -0.06 0.0 rpy=0 0 0 -> xyz=0.0 -0.1 0.0 rpy=0 0 0
- joint th_7: axis -1.0 0.0 0.0 -> 1.0 -0.0 -0.0; origin xyz=0.0 -0.06 0.0 rpy=0 0 0 -> xyz=0.0 -0.1 0.0 rpy=0 0 0
- joint th_8: axis 1.0 0.0 0.0 -> -1.0 -0.0 0.0; origin xyz=0.0 -0.06 0.0 rpy=0 0 0 -> xyz=0.0 -0.1 0.0 rpy=0 0 0
